File: schematics/nixie-clock/nixie-clock.kicad_sch (KiCad schematic)
At the start: 45 parts, among them J1 Barrel_Jack_Switch, J2 Conn_02x03_Odd_Even, J3 Screw_Terminal_01x02, J4 Screw_Terminal_01x02, Q1 MJE13007, Q2 MJE13007, SW1 SW_Push, SW2 SW_Push, SW3 SW_Push, U1 LM317_TO-220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

Commit message: schematic: added mounting holes
Parts:
- added H1, H2, H3, H4: MountingHole, MountingHole:MountingHole_3mm, symbol Mechanical:MountingHole
Other:
- note added: "Mounting holes"
Changed lines of the file:
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@@
     (stroke (width 0) (type default) (color 0 0 0 0))
   )
+  (polyline (pts (xy 289.56 203.2) (xy 289.56 231.14))
+    (stroke (width 0) (type default) (color 0 0 0 0))
+  )
   (polyline (pts (xy 123.19 59.69) (xy 154.94 59.69))
     (stroke (width 0) (type default) (color 0 0 0 0))
@@
     (stroke (width 0) (type default) (color 0 0 0 0))
   )
+  (polyline (pts (xy 320.04 203.2) (xy 289.56 203.2))
+    (stroke (width 0) (type default) (color 0 0 0 0))
+  )
   (polyline (pts (xy 133.35 105.41) (xy 133.35 144.78))
     (stroke (width 0) (type default) (color 0 0 0 0))
@@
     (stroke (width 0) (type default) (color 0 0 0 0))
   )
+  (polyline (pts (xy 289.56 231.14) (xy 320.04 231.14))
+    (stroke (width 0) (type default) (color 0 0 0 0))
+  )
   (wire (pts (xy 237.49 58.42) (xy 254 58.42))
     (stroke (width 0) (type default) (color 0 0 0 0))
@@
     (stroke (width 0) (type default) (color 0 0 0 0))
   )
+  (polyline (pts (xy 320.04 203.2) (xy 320.04 231.14))
+    (stroke (width 0) (type default) (color 0 0 0 0))
+  )
   (polyline (pts (xy 151.13 118.11) (xy 151.13 125.73))
     (stroke (width 0) (type default) (color 0 0 0 0))
@@
     (effects (font (size 1.27 1.27) bold) (justify left bottom))
   )
+  (text "Mounting holes" (at 297.18 207.01 0)
+    (effects (font (size 1.27 1.27) (thickness 0.254) bold) (justify left bottom))
+  )
   (label "N3B" (at 374.65 220.98 0)
     (effects (font (size 1.27 1.27)) (justify left bottom))
@@
     (pin "9")
   )
+  (symbol (lib_id "Mechanical:MountingHole") (at 295.91 227.33 0) (unit 1)
+    (in_bom yes) (on_board yes) (fields_autoplaced)
+    (property "Reference" "H4" (id 0) (at 298.45 226.0599 0)
+      (effects (font (size 1.27 1.27)) (justify left))
+    )
+    (property "Value" "MountingHole" (id 1) (at 298.45 228.5999 0)
+      (effects (font (size 1.27 1.27)) (justify left))
+    )
+    (property "Footprint" "MountingHole:MountingHole_3mm" (id 2) (at 295.91 227.33 0)
+      (effects (font (size 1.27 1.27)) hide)
+    )
+    (property "Datasheet" "~" (id 3) (at 295.91 227.33 0)
+      (effects (font (size 1.27 1.27)) hide)
+    )
+  )
   (symbol (lib_id "nixies-us:IN-1") (at 264.16 109.22 0) (unit 1)
     (in_bom yes) (on_board yes) (fields_autoplaced)
@@
     (pin "A")
   )
+  (symbol (lib_id "Mechanical:MountingHole") (at 295.91 217.17 0) (unit 1)
+    (in_bom yes) (on_board yes) (fields_autoplaced)
+    (property "Reference" "H2" (id 0) (at 298.45 215.8999 0)
+      (effects (font (size 1.27 1.27)) (justify left))
+    )
+    (property "Value" "MountingHole" (id 1) (at 298.45 218.4399 0)
+      (effects (font (size 1.27 1.27)) (justify left))
+    )
+    (property "Footprint" "MountingHole:MountingHole_3mm" (id 2) (at 295.91 217.17 0)
+      (effects (font (size 1.27 1.27)) hide)
+    )
+    (property "Datasheet" "~" (id 3) (at 295.91 217.17 0)
+      (effects (font (size 1.27 1.27)) hide)
+    )
+  )
   (symbol (lib_id "CustomComponents:K155NA1") (at 212.09 107.95 0) (unit 1)
     (in_bom yes) (on_board yes) (fields_autoplaced)
@@
     (pin "1")
   )
+  (symbol (lib_id "Mechanical:MountingHole") (at 295.91 222.25 0) (unit 1)
+    (in_bom yes) (on_board yes) (fields_autoplaced)
+    (property "Reference" "H3" (id 0) (at 298.45 220.9799 0)
+      (effects (font (size 1.27 1.27)) (justify left))
+    )
+    (property "Value" "MountingHole" (id 1) (at 298.45 223.5199 0)
+      (effects (font (size 1.27 1.27)) (justify left))
+    )
+    (property "Footprint" "MountingHole:MountingHole_3mm" (id 2) (at 295.91 222.25 0)
+      (effects (font (size 1.27 1.27)) hide)
+    )
+    (property "Datasheet" "~" (id 3) (at 295.91 222.25 0)
+      (effects (font (size 1.27 1.27)) hide)
+    )
+  )
   (symbol (lib_id "Switch:SW_Push") (at 106.68 130.81 0) (unit 1)
     (in_bom yes) (on_board yes)
@@
     (pin "2")
   )
+  (symbol (lib_id "Mechanical:MountingHole") (at 295.91 212.09 0) (unit 1)
+    (in_bom yes) (on_board yes) (fields_autoplaced)
+    (property "Reference" "H1" (id 0) (at 298.45 210.8199 0)
+      (effects (font (size 1.27 1.27)) (justify left))
+    )
+    (property "Value" "MountingHole" (id 1) (at 298.45 213.3599 0)
+      (effects (font (size 1.27 1.27)) (justify left))
+    )
+    (property "Footprint" "MountingHole:MountingHole_3mm" (id 2) (at 295.91 212.09 0)
+      (effects (font (size 1.27 1.27)) hide)
+    )
+    (property "Datasheet" "~" (id 3) (at 295.91 212.09 0)
+      (effects (font (size 1.27 1.27)) hide)
+    )
+  )
   (symbol (lib_name "+5V_2") (lib_id "power:+5V") (at 53.34 114.3 0) (unit 1)
     (in_bom yes) (on_board yes)
@@
       (reference "C8") (unit 1) (value "100n") (footprint "Capacitor_SMD:C_0805_2012Metric_Pad1.18x1.45mm_HandSolder")
     )
+    (path "/d95d255b-eaf0-4763-9d7b-013d7a25717c"
+      (reference "H1") (unit 1) (value "MountingHole") (footprint "MountingHole:MountingHole_3mm")
+    )
+    (path "/627c102b-8ccf-4595-bb79-ea23cb1dde17"
+      (reference "H2") (unit 1) (value "MountingHole") (footprint "MountingHole:MountingHole_3mm")
+    )
+    (path "/c95a5be1-89df-4286-b806-21dd9a5ddf46"
+      (reference "H3") (unit 1) (value "MountingHole") (footprint "MountingHole:MountingHole_3mm")
+    )
+    (path "/2af466aa-a205-4ad0-9e04-0a05e9fe9098"
+      (reference "H4") (unit 1) (value "MountingHole") (footprint "MountingHole:MountingHole_3mm")
+    )
     (path "/a8bcdb0a-cd57-401c-aa12-e9b2745ef5d4"
