File: schematics/nixie-clock/nixie-clock.kicad_pcb (KiCad board)
At the start: 2 copper layers, 320 x 168.9 mm, 49 parts, among them J1 Barrel_Jack_Switch, J2 Conn_02x03_Odd_Even, J3 Screw_Terminal_01x02, J4 Screw_Terminal_01x02, Q1 MJE13007, Q2 MJE13007, SW1 SW_Push, SW2 SW_Push, SW3 SW_Push, U1 LM317_TO-220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

Commit message: schematic: added inter-panel connection
Parts:
- added H5: MountingHole, MountingHole:MountingHole_3mm, F.Cu at (368.4, 120.7)
- added H6: MountingHole, MountingHole:MountingHole_3mm, F.Cu at (375.9, 120.7)
- added H7: MountingHole, MountingHole:MountingHole_3mm, F.Cu at (384.2, 116.3)
- added H8: MountingHole, MountingHole:MountingHole_3mm, F.Cu at (367.0, 106.7)
- added J5: Screw_Terminal_01x03, TerminalBlock_Phoenix:TerminalBlock_Phoenix_MKDS-1,5-3_1x03_P5.00mm_Horizontal, F.Cu at (340.4, 158.8)
- added J6: Conn_01x03, Connector_PinHeader_2.54mm:PinHeader_1x03_P2.54mm_Horizontal, F.Cu at (92.7, 145.3)
- added J7: Conn_01x03, Connector_PinHeader_2.54mm:PinHeader_1x03_P2.54mm_Horizontal, F.Cu at (102.9, 36.1)
- added J8: Conn_01x04, Connector_PinHeader_2.54mm:PinHeader_1x03_P2.54mm_Horizontal, F.Cu at (144.2, 188.0)
- added J9: Screw_Terminal_01x03, TerminalBlock_Phoenix:TerminalBlock_Phoenix_MKDS-1,5-3_1x03_P5.00mm_Horizontal, F.Cu at (340.4, 167.9)
- added R11: 33k, Resistor_THT:R_Axial_DIN0309_L9.0mm_D3.2mm_P12.70mm_Horizontal, F.Cu at (463.7, 310.4)
- added R12: 33k, Resistor_THT:R_Axial_DIN0309_L9.0mm_D3.2mm_P12.70mm_Horizontal, F.Cu at (404.9, 305.1)
- added R13: 33k, Resistor_THT:R_Axial_DIN0309_L9.0mm_D3.2mm_P12.70mm_Horizontal, F.Cu at (421.9, 286.1)
- added R14: 33k, Resistor_THT:R_Axial_DIN0309_L9.0mm_D3.2mm_P12.70mm_Horizontal, F.Cu at (404.9, 309.8)
- added R15: 33k, Resistor_THT:R_Axial_DIN0309_L9.0mm_D3.2mm_P12.70mm_Horizontal, F.Cu at (487.7, 308.7)
- added R16: 33k, Resistor_THT:R_Axial_DIN0309_L9.0mm_D3.2mm_P12.70mm_Horizontal, F.Cu at (421.9, 290.9)
- added R17: 33k, Resistor_THT:R_Axial_DIN0309_L9.0mm_D3.2mm_P12.70mm_Horizontal, F.Cu at (196.8, 112.9)
- added R18: 33k, Resistor_THT:R_Axial_DIN0309_L9.0mm_D3.2mm_P12.70mm_Horizontal, F.Cu at (196.8, 116.7)
- BT1: moved to B.Cu
- moved R7 218.8 mm to (266.7, 63.5)
- moved U3 180.7 mm to (7.62, 43.2)
- moved U5 180.7 mm to (-20.3, 31.7)
- moved U6 180.7 mm to (17.8, 31.7)
- moved R8 175.6 mm to (-49.1, 110.1)
- moved R6 175.6 mm to (-49.3, 113.0)
- moved J3 162.6 mm to (73.7, 215.2), turned to 90 degrees
- moved C8 111.0 mm to (355.6, 233.7)
- moved C7 111.0 mm to (335.4, 233.7)
- moved SW2 111.0 mm to (337.9, 223.5)
- moved SW3 111.0 mm to (358.1, 223.5)
- moved BZ1 107.3 mm to (55.9, 151.1), turned to -90 degrees
- moved J4 98.7 mm to (125.1, 210.2), turned to -90 degrees
- moved SW1 95.7 mm to (73.9, 174.9), turned to 90 degrees
- moved C2 94.5 mm to (97.6, 200.5), turned to -90 degrees
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Connections:
- net RTC_SCL renamed SCL
- net RTC_SDA renamed SDA
- J4 pad 2: HIGH VOLTAGE -> BOOSTER OUT
- N1 pad A: HIGH VOLTAGE -> Net-(N1-PadA)
- N2 pad A: HIGH VOLTAGE -> Net-(N2-PadA)
- N3 pad A: HIGH VOLTAGE -> Net-(N3-PadA)
- N4 pad A: HIGH VOLTAGE -> Net-(N4-PadA)
- U2 pad 23: SER1 -> SER1_CON
- U2 pad 24: SRCLK -> SRCLK_CON
- U2 pad 25: RCLK -> RCLK_CON
Routing:
- net +5V: track 5.89 -> 123.8 mm
- net SDA: track 0.00 -> 69.3 mm
- net SCL: track 0.00 -> 66.3 mm, vias 0 -> 1
- net MOSI: track 0.00 -> 28.0 mm
- net RST: track 0.00 -> 27.2 mm
- net MISO: track 0.00 -> 26.0 mm
- net Net-(BT1-Pad1): track 0.00 -> 21.7 mm
- net SCK: track 0.00 -> 20.9 mm
- net GND: track 0.00 -> 11.7 mm
- net Crystal1: track 0.00 -> 11.1 mm
- net Crystal2: track 0.00 -> 11.0 mm
- net Net-(U9-Pad2): track 0.00 -> 2.50 mm
- net Net-(U9-Pad1): track 0.00 -> 2.49 mm
- net Net-(R1-Pad2): track 8.10 -> 6.50 mm
- added copper zone on F.Cu, net GND
Other:
- board size 320 x 168.9 mm -> 170.2 x 171.4 mm

Commit message: pcb: placed elements on main board, added mounting holes
Parts:
- removed the J6 at (92.7, 145.3)
- removed J9: Screw_Terminal_01x03, TerminalBlock_Phoenix:TerminalBlock_Phoenix_MKDS-1,5-3_1x03_P5.00mm_Horizontal
- added H10: MountingHole, MountingHole:MountingHole_3mm, F.Cu at (135.3, 128.3)
- added H11: MountingHole, MountingHole:MountingHole_3mm, F.Cu at (161.9, 128.3)
- added H12: MountingHole, MountingHole:MountingHole_3mm, F.Cu at (161.9, 54.6)
- added H9: MountingHole, MountingHole:MountingHole_3mm, F.Cu at (135.3, 54.6)
- BZ1, J2, R1, SW1: moved to B.Cu
- C7, C8, Y2: moved to F.Cu
- J3: renamed from J8; footprint Connector_PinHeader_2.54mm:PinHeader_1x03_P2.54mm_Horizontal -> Connector_PinHeader_2.54mm:PinHeader_1x04_P2.54mm_Vertical
- J4: value Screw_Terminal_01x02 -> Conn_01x07; footprint TerminalBlock_Phoenix:TerminalBlock_Phoenix_MKDS-1,5-2_1x02_P5.00mm_Horizontal -> Connector_PinHeader_2.54mm:PinHeader_1x07_P2.54mm_Horizontal
- J5: value Screw_Terminal_01x03 -> Conn_01x07; footprint TerminalBlock_Phoenix:TerminalBlock_Phoenix_MKDS-1,5-3_1x03_P5.00mm_Horizontal -> Connector_PinHeader_2.54mm:PinHeader_1x07_P2.54mm_Horizontal; moved to B.Cu
- J7: value Conn_01x03 -> Screw_Terminal_01x02; footprint Connector_PinHeader_2.54mm:PinHeader_1x03_P2.54mm_Horizontal -> TerminalBlock_Phoenix:TerminalBlock_Phoenix_MKDS-1,5-2_1x02_P5.00mm_Horizontal; moved to B.Cu
- SW2, SW3: footprint Button_Switch_Keyboard:SW_Cherry_MX_1.00u_PCB -> Button_Switch_THT:SW_PUSH_6mm_H13mm; moved to B.Cu
- moved R11 436.3 mm to (73.7, 114.9), turned to -90 degrees
- moved R15 388.3 mm to (151.1, 114.9), turned to -90 degrees
- moved R12 385.2 mm to (69.8, 114.9), turned to -90 degrees
- moved R13 360.4 mm to (104.8, 114.9), turned to -90 degrees
- moved R14 354.6 mm to (108.6, 114.9), turned to -90 degrees
- moved H6 330.4 mm to (60.3, 218.4)
- moved R16 319.7 mm to (154.9, 114.9), turned to -90 degrees
- moved H1 315.8 mm to (60.3, 54.6)
- moved H5 309.0 mm to (60.3, 144.8)
- moved H2 299.3 mm to (60.3, 128.3)
- moved SW3 279.2 mm to (85.4, 163.8), turned to -90 degrees
- moved C8 276.1 mm to (87.6, 167.0), turned to 180 degrees
- moved J5 274.9 mm to (85.7, 55.2), turned to 90 degrees
- moved C7 264.3 mm to (79.7, 167.0)
- moved SW2 261.5 mm to (81.9, 170.3), turned to 90 degrees
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- renumbered J3 to J6
Connections:
- J4 pad 1: GND -> +5V
- J4 pad 2: BOOSTER OUT -> SER1_CON
- J5 pad 1: BOOSTER OUT -> GNDA
- J5 pad 2: +5V -> BULB2
- J5 pad 3: GND -> BULB1
- J7 pad 1: SRCLK -> unconnected-(J7-Pad1)
- J7 pad 2: RCLK -> HIGH VOLTAGE
- Q1 pad 3: GND -> GNDA
- Q2 pad 3: GND -> GNDA
- U2 pad 2: BULB1 -> BULB1_CON
- U2 pad 3: BULB2 -> BULB2_CON
- U3 pad 10: +5V -> +5VA
- U3 pad 13: +5V -> +5VA
- U3 pad 16: +5V -> +5VA
- U3 pad 8: GND -> GNDA
- U4 pad 10: +5V -> +5VA
- U4 pad 13: +5V -> +5VA
- U4 pad 16: +5V -> +5VA
- U4 pad 8: GND -> GNDA
- U5 pad 12: GND -> GNDA
- U5 pad 5: +5V -> +5VA
- U6 pad 12: GND -> GNDA
- U6 pad 5: +5V -> +5VA
- U7 pad 12: GND -> GNDA
- U7 pad 5: +5V -> +5VA
- U8 pad 12: GND -> GNDA
- U8 pad 5: +5V -> +5VA
- Y2 pad 1: Net-(U9-Pad2) -> Net-(U9-Pad1)
- Y2 pad 2: Net-(U9-Pad1) -> Net-(U9-Pad2)
Routing:
- net +5V: track 123.8 -> 0.00 mm
- net SDA: track 69.3 -> 0.00 mm
- net SCL: track 66.3 -> 0.00 mm
- net MOSI: track 28.0 -> 0.00 mm
- net RST: track 27.2 -> 0.00 mm
- net MISO: track 26.0 -> 0.00 mm
- net Net-(BT1-Pad1): track 21.7 -> 0.00 mm
- net SCK: track 20.9 -> 0.00 mm
- net GND: track 11.7 -> 0.00 mm
- net Crystal1: track 11.1 -> 0.00 mm
- net Crystal2: track 11.0 -> 0.00 mm
- net Net-(R1-Pad2): track 6.50 -> 0.00 mm
- net Net-(U9-Pad2): track 2.50 -> 0.00 mm
- net Net-(U9-Pad1): track 2.49 -> 0.00 mm
- removed copper zone on F.Cu, net GND
Other:
- board size 170.2 x 171.4 mm -> 184.1 x 171.4 mm
- board text added: "5V"
- board text added: "GND"
- board text added: "ICSP"
- board text added: "MISO"
- board text added: "MOSI"
- board text added: "RST"
- board text added: "SCK"
- board text added: "SCL"
- board text added: "SDA"

Commit message: pcb: finished, tweaks to be done
Parts:
- R11, R12, R13, R14, R15, R16, R17, R18: footprint Resistor_THT:R_Axial_DIN0309_L9.0mm_D3.2mm_P12.70mm_Horizontal -> Resistor_SMD:R_1206_3216Metric_Pad1.30x1.75mm_HandSolder
- moved R13 10.0 mm to (114.3, 118.1)
- moved R15 9.44 mm to (160.0, 118.1)
- moved R14 8.84 mm to (116.8, 118.1)
- moved R16 8.26 mm to (162.6, 118.1)
- moved R17 7.67 mm to (198.1, 118.1)
- moved BZ1 7.61 mm to (131.3, 183.5), turned to 90 degrees
- moved R12 7.10 mm to (76.2, 118.1)
- moved R18 6.54 mm to (200.7, 118.1)
- moved R11 5.99 mm to (78.7, 118.1)
- moved R1 5.72 mm to (64.1, 188.6)
- moved C2 4.69 mm to (77.5, 193.3), turned to -90 degrees
- moved R4 4.45 mm to (114.1, 193.0)
- moved R5 4.45 mm to (116.0, 193.0)
- moved C3 1.91 mm to (94.6, 193.0)
- moved C4 1.91 mm to (99.5, 193.0)
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Routing:
- net +5VA: track 0.00 -> 196.5 mm
- net +5V: track 0.00 -> 172.8 mm
- net HIGH VOLTAGE: track 0.00 -> 155.8 mm
- net RCLK: track 0.00 -> 130.4 mm, vias 0 -> 1
- net SRCLK: track 0.00 -> 126.3 mm, vias 0 -> 4
- net BULB1: track 0.00 -> 78.1 mm, vias 0 -> 1
- net SER2: track 0.00 -> 74.6 mm
- net SCL: track 0.00 -> 74.0 mm, vias 1 -> 2
- net SDA: track 0.00 -> 72.4 mm, vias 0 -> 1
- net BULB2_CON: track 0.00 -> 68.9 mm
- net BULB2: track 0.00 -> 67.0 mm, vias 0 -> 1
- net RST: track 0.00 -> 63.3 mm
- net Net-(N3-Pad2): track 0.00 -> 62.6 mm
- net Net-(N2-Pad2): track 0.00 -> 61.1 mm
- net Net-(N4-Pad2): track 0.00 -> 61.1 mm
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- added copper zone on F.Cu, net GND
- added copper zone on F.Cu, net GNDA
